Commit message: backup_attache

File: ros2_iiwa/iiwa_description/urdf/iiwa1.urdf.xacro (robot description, xacro)
@@ -38,5 +38,5 @@
         <origin xyz="0 0 0.01" rpy="0 0 0"/>
         <geometry><cylinder radius="0.06" length="0.36"/></geometry>
-      </collision>-
+      </collision>
       <inertial>
         <origin xyz="0 0 0.01" rpy="0 0 0"/>
@@ -185,4 +185,37 @@
       <parent link="${prefix}link_7"/><child link="${prefix}tool0"/>
     </joint>
+    <link name="${prefix}vacuum_gripper_link">
+      <visual>
+        <origin xyz="0 0 0.01" rpy="0 0 0"/>
+        <geometry><cylinder radius="0.04" length="0.02"/></geometry>
+        <material name="Black"><color rgba="0.1 0.1 0.1 1"/></material>
+      </visual>
+      <collision name="${prefix}vacuum_gripper_collision">
+        <origin xyz="0 0 0.01" rpy="0 0 0"/>
+        <geometry><cylinder radius="0.04" length="0.02"/></geometry>
+      </collision>
+      <inertial>
+        <mass value="0.1"/>
+        <inertia ixx="0.0001" ixy="0" ixz="0" iyy="0.0001" iyz="0" izz="0.0001"/>
+      </inertial>
+    </link>
+    <joint name="${prefix}vacuum_gripper_joint" type="fixed">
+      <parent link="${prefix}tool0"/>
+      <child link="${prefix}vacuum_gripper_link"/>
+      <origin xyz="0 0 0" rpy="0 0 0"/>
+    </joint>
+    <gazebo reference="${prefix}vacuum_gripper_link">
+      <sensor name="suction_contact" type="contact">
+        <contact>
+          <collision>${prefix}vacuum_gripper_collision</collision>
+        </contact>
+        <update_rate>30</update_rate>
+        <always_on>true</always_on>
+      </sensor>
+    </gazebo>
+    <gazebo reference="${prefix}vacuum_gripper_joint">
+      <preserveFixedJoint>true</preserveFixedJoint>
+      <disableFixedJointLumping>true</disableFixedJointLumping>
+    </gazebo>
   </xacro:macro>
   <link name="world"/>
@@ -201,4 +234,26 @@
   </ros2_control>
   <gazebo>
+    <plugin filename="libignition-gazebo-detachable-joint-system.so"
+            name="ignition::gazebo::systems::DetachableJoint">
+      <parent_link>iiwa_vacuum_gripper_link</parent_link>
+      <child_model>package</child_model>
+      <child_link>package_link</child_link>
+      <output_topic>/iiwa1/gripper/state_package</output_topic>
+      <detach_topic>/iiwa1/gripper/detach_package</detach_topic>
+      <attach_topic>/iiwa1/gripper/attach_package</attach_topic>
+    </plugin>
+  </gazebo>
+  <gazebo>
+    <plugin filename="libignition-gazebo-detachable-joint-system.so"
+            name="ignition::gazebo::systems::DetachableJoint">
+      <parent_link>iiwa_vacuum_gripper_link</parent_link>
+      <child_model>package2</child_model>
+      <child_link>package2_link</child_link>
+      <output_topic>/iiwa1/gripper/state_package2</output_topic>
+      <detach_topic>/iiwa1/gripper/detach_package2</detach_topic>
+      <attach_topic>/iiwa1/gripper/attach_package2</attach_topic>
+    </plugin>
+  </gazebo>
+  <gazebo>
     <plugin filename="libgz_ros2_control-system.so" name="gz_ros2_control::GazeboSimROS2ControlPlugin">
       <parameters>$(find iiwa_description)/config/iiwa1_controllers.yaml</parameters>

File: ros2_iiwa/iiwa_description/urdf/iiwa2.urdf.xacro (robot description, xacro)
@@ -194,4 +194,37 @@
         </camera>
       </sensor>
+    </gazebo>
+     <link name="${prefix}vacuum_gripper_link">
+      <visual>
+        <origin xyz="0 0 0.01" rpy="0 0 0"/>
+        <geometry><cylinder radius="0.04" length="0.02"/></geometry>
+        <material name="Black"><color rgba="0.1 0.1 0.1 1"/></material>
+      </visual>
+      <collision name="${prefix}vacuum_gripper_collision">
+        <origin xyz="0 0 0.01" rpy="0 0 0"/>
+        <geometry><cylinder radius="0.04" length="0.02"/></geometry>
+      </collision>
+      <inertial>
+        <mass value="0.1"/>
+        <inertia ixx="0.0001" ixy="0" ixz="0" iyy="0.0001" iyz="0" izz="0.0001"/>
+      </inertial>
+    </link>
+    <joint name="${prefix}vacuum_gripper_joint" type="fixed">
+      <parent link="${prefix}tool0"/>
+      <child link="${prefix}vacuum_gripper_link"/>
+      <origin xyz="0 0 0" rpy="0 0 0"/>
+    </joint>
+    <gazebo reference="${prefix}vacuum_gripper_link">
+      <sensor name="suction_contact" type="contact">
+        <contact>
+          <collision>${prefix}vacuum_gripper_collision</collision>
+        </contact>
+        <update_rate>30</update_rate>
+        <always_on>true</always_on>
+      </sensor>
+    </gazebo>
+    <gazebo reference="${prefix}vacuum_gripper_joint">
+      <preserveFixedJoint>true</preserveFixedJoint>
+      <disableFixedJointLumping>true</disableFixedJointLumping>
     </gazebo>
   </xacro:macro>
@@ -211,4 +244,26 @@
   </ros2_control>
   <gazebo>
+    <plugin filename="libignition-gazebo-detachable-joint-system.so"
+            name="ignition::gazebo::systems::DetachableJoint">
+      <parent_link>iiwa2_vacuum_gripper_link</parent_link>
+      <child_model>package</child_model>
+      <child_link>package_link</child_link>
+      <output_topic>/iiwa2/gripper/state_package</output_topic>
+      <detach_topic>/iiwa2/gripper/detach_package</detach_topic>
+      <attach_topic>/iiwa2/gripper/attach_package</attach_topic>
+    </plugin>
+  </gazebo>
+  <gazebo>
+    <plugin filename="libignition-gazebo-detachable-joint-system.so"
+            name="ignition::gazebo::systems::DetachableJoint">
+      <parent_link>iiwa2_vacuum_gripper_link</parent_link>
+      <child_model>package2</child_model>
+      <child_link>package2_link</child_link>
+      <output_topic>/iiwa2/gripper/state_package2</output_topic>
+      <detach_topic>/iiwa2/gripper/detach_package2</detach_topic>
+      <attach_topic>/iiwa2/gripper/attach_package2</attach_topic>
+    </plugin>
+  </gazebo>
+  <gazebo>
     <plugin filename="libgz_ros2_control-system.so" name="gz_ros2_control::GazeboSimROS2ControlPlugin">
       <parameters>$(find iiwa_description)/config/iiwa2_controllers.yaml</parameters>

Commit message: prisco effect

File: ros2_iiwa/iiwa_description/urdf/iiwa1.urdf.xacro (robot description, xacro)
@@ -260,5 +260,8 @@
       <robot_param>robot_description</robot_param>
       <robot_param_node>robot_state_publisher</robot_param_node>
-      <ros><namespace>iiwa</namespace></ros>
+      <ros>
+        <namespace>iiwa</namespace>
+        <remapping>controller_manager/robot_description:=robot_description</remapping>
+      </ros>
     </plugin>
   </gazebo>

File: ros2_iiwa/iiwa_description/urdf/iiwa2.urdf.xacro (robot description, xacro)
@@ -238,11 +238,11 @@
     <param name="use_sim_time">true</param>
   </hardware>
-    <joint name="iiwa2_joint_a1"><command_interface name="velocity"/><state_interface name="position"/><state_interface name="velocity"/></joint>
-    <joint name="iiwa2_joint_a2"><command_interface name="velocity"/><state_interface name="position"/><state_interface name="velocity"/></joint>
-    <joint name="iiwa2_joint_a3"><command_interface name="velocity"/><state_interface name="position"/><state_interface name="velocity"/></joint>
-    <joint name="iiwa2_joint_a4"><command_interface name="velocity"/><state_interface name="position"/><state_interface name="velocity"/></joint>
-    <joint name="iiwa2_joint_a5"><command_interface name="velocity"/><state_interface name="position"/><state_interface name="velocity"/></joint>
-    <joint name="iiwa2_joint_a6"><command_interface name="velocity"/><state_interface name="position"/><state_interface name="velocity"/></joint>
-    <joint name="iiwa2_joint_a7"><command_interface name="velocity"/><state_interface name="position"/><state_interface name="velocity"/></joint>
+    <joint name="iiwa2_joint_a1"><command_interface name="position"/><state_interface name="position"/><state_interface name="velocity"/></joint>
+    <joint name="iiwa2_joint_a2"><command_interface name="position"/><state_interface name="position"/><state_interface name="velocity"/></joint>
+    <joint name="iiwa2_joint_a3"><command_interface name="position"/><state_interface name="position"/><state_interface name="velocity"/></joint>
+    <joint name="iiwa2_joint_a4"><command_interface name="position"/><state_interface name="position"/><state_interface name="velocity"/></joint>
+    <joint name="iiwa2_joint_a5"><command_interface name="position"/><state_interface name="position"/><state_interface name="velocity"/></joint>
+    <joint name="iiwa2_joint_a6"><command_interface name="position"/><state_interface name="position"/><state_interface name="velocity"/></joint>
+    <joint name="iiwa2_joint_a7"><command_interface name="position"/><state_interface name="position"/><state_interface name="velocity"/></joint>
   </ros2_control>
   <gazebo>
