Commit message: detection

File: ros2_iiwa/iiwa_description/urdf/iiwa2.urdf.xacro (robot description, xacro)
@@ -183,5 +183,5 @@
     </joint>
     <joint name="${prefix}camera_joint" type="fixed">
-      <parent link="${prefix}tool0"/><child link="${prefix}camera_link"/><origin xyz="0 0 0.02" rpy="0 0 0"/>
+      <parent link="${prefix}tool0"/><child link="${prefix}camera_link"/><origin xyz="0 0 0.02" rpy="0 -1.57 -1.57"/>
     </joint>
     <gazebo reference="${prefix}camera_link">
@@ -235,11 +235,11 @@
   <ros2_control name="iiwa2_hardware" type="system">
     <hardware><plugin>gz_ros2_control/GazeboSimSystem</plugin></hardware>
-    <joint name="iiwa2_joint_a1"><command_interface name="position"/><state_interface name="position"/><state_interface name="velocity"/></joint>
-    <joint name="iiwa2_joint_a2"><command_interface name="position"/><state_interface name="position"/><state_interface name="velocity"/></joint>
-    <joint name="iiwa2_joint_a3"><command_interface name="position"/><state_interface name="position"/><state_interface name="velocity"/></joint>
-    <joint name="iiwa2_joint_a4"><command_interface name="position"/><state_interface name="position"/><state_interface name="velocity"/></joint>
-    <joint name="iiwa2_joint_a5"><command_interface name="position"/><state_interface name="position"/><state_interface name="velocity"/></joint>
-    <joint name="iiwa2_joint_a6"><command_interface name="position"/><state_interface name="position"/><state_interface name="velocity"/></joint>
-    <joint name="iiwa2_joint_a7"><command_interface name="position"/><state_interface name="position"/><state_interface name="velocity"/></joint>
+    <joint name="iiwa2_joint_a1"><command_interface name="position"/><command_interface name="velocity"/><state_interface name="position"/><state_interface name="velocity"/></joint>
+    <joint name="iiwa2_joint_a2"><command_interface name="position"/><command_interface name="velocity"/><state_interface name="position"/><state_interface name="velocity"/></joint>
+    <joint name="iiwa2_joint_a3"><command_interface name="position"/><command_interface name="velocity"/><state_interface name="position"/><state_interface name="velocity"/></joint>
+    <joint name="iiwa2_joint_a4"><command_interface name="position"/><command_interface name="velocity"/><state_interface name="position"/><state_interface name="velocity"/></joint>
+    <joint name="iiwa2_joint_a5"><command_interface name="position"/><command_interface name="velocity"/><state_interface name="position"/><state_interface name="velocity"/></joint>
+    <joint name="iiwa2_joint_a6"><command_interface name="position"/><command_interface name="velocity"/><state_interface name="position"/><state_interface name="velocity"/></joint>
+    <joint name="iiwa2_joint_a7"><command_interface name="position"/><command_interface name="velocity"/><state_interface name="position"/><state_interface name="velocity"/></joint>
   </ros2_control>
   <gazebo>

Commit message: velocity

File: ros2_iiwa/iiwa_description/urdf/iiwa2.urdf.xacro (robot description, xacro)
@@ -234,12 +234,15 @@
   </xacro:iiwa2_macro>
   <ros2_control name="iiwa2_hardware" type="system">
-    <hardware><plugin>gz_ros2_control/GazeboSimSystem</plugin></hardware>
-    <joint name="iiwa2_joint_a1"><command_interface name="position"/><command_interface name="velocity"/><state_interface name="position"/><state_interface name="velocity"/></joint>
-    <joint name="iiwa2_joint_a2"><command_interface name="position"/><command_interface name="velocity"/><state_interface name="position"/><state_interface name="velocity"/></joint>
-    <joint name="iiwa2_joint_a3"><command_interface name="position"/><command_interface name="velocity"/><state_interface name="position"/><state_interface name="velocity"/></joint>
-    <joint name="iiwa2_joint_a4"><command_interface name="position"/><command_interface name="velocity"/><state_interface name="position"/><state_interface name="velocity"/></joint>
-    <joint name="iiwa2_joint_a5"><command_interface name="position"/><command_interface name="velocity"/><state_interface name="position"/><state_interface name="velocity"/></joint>
-    <joint name="iiwa2_joint_a6"><command_interface name="position"/><command_interface name="velocity"/><state_interface name="position"/><state_interface name="velocity"/></joint>
-    <joint name="iiwa2_joint_a7"><command_interface name="position"/><command_interface name="velocity"/><state_interface name="position"/><state_interface name="velocity"/></joint>
+    <hardware>
+    <plugin>gz_ros2_control/GazeboSimSystem</plugin>
+    <param name="use_sim_time">true</param>
+  </hardware>
+    <joint name="iiwa2_joint_a1"><command_interface name="velocity"/><state_interface name="position"/><state_interface name="velocity"/></joint>
+    <joint name="iiwa2_joint_a2"><command_interface name="velocity"/><state_interface name="position"/><state_interface name="velocity"/></joint>
+    <joint name="iiwa2_joint_a3"><command_interface name="velocity"/><state_interface name="position"/><state_interface name="velocity"/></joint>
+    <joint name="iiwa2_joint_a4"><command_interface name="velocity"/><state_interface name="position"/><state_interface name="velocity"/></joint>
+    <joint name="iiwa2_joint_a5"><command_interface name="velocity"/><state_interface name="position"/><state_interface name="velocity"/></joint>
+    <joint name="iiwa2_joint_a6"><command_interface name="velocity"/><state_interface name="position"/><state_interface name="velocity"/></joint>
+    <joint name="iiwa2_joint_a7"><command_interface name="velocity"/><state_interface name="position"/><state_interface name="velocity"/></joint>
   </ros2_control>
   <gazebo>

Commit message: primo_commit

File: ros2_iiwa/iiwa_description/urdf/iiwa2.urdf.xacro (robot description, xacro)
@@ -238,11 +238,11 @@
     <param name="use_sim_time">true</param>
   </hardware>
-    <joint name="iiwa2_joint_a1"><command_interface name="position"/><state_interface name="position"/><state_interface name="velocity"/></joint>
-    <joint name="iiwa2_joint_a2"><command_interface name="position"/><state_interface name="position"/><state_interface name="velocity"/></joint>
-    <joint name="iiwa2_joint_a3"><command_interface name="position"/><state_interface name="position"/><state_interface name="velocity"/></joint>
-    <joint name="iiwa2_joint_a4"><command_interface name="position"/><state_interface name="position"/><state_interface name="velocity"/></joint>
-    <joint name="iiwa2_joint_a5"><command_interface name="position"/><state_interface name="position"/><state_interface name="velocity"/></joint>
-    <joint name="iiwa2_joint_a6"><command_interface name="position"/><state_interface name="position"/><state_interface name="velocity"/></joint>
-    <joint name="iiwa2_joint_a7"><command_interface name="position"/><state_interface name="position"/><state_interface name="velocity"/></joint>
+    <joint name="iiwa2_joint_a1"><command_interface name="position"/><command_interface name="velocity"/><state_interface name="position"/><state_interface name="velocity"/></joint>
+    <joint name="iiwa2_joint_a2"><command_interface name="position"/><command_interface name="velocity"/><state_interface name="position"/><state_interface name="velocity"/></joint>
+    <joint name="iiwa2_joint_a3"><command_interface name="position"/><command_interface name="velocity"/><state_interface name="position"/><state_interface name="velocity"/></joint>
+    <joint name="iiwa2_joint_a4"><command_interface name="position"/><command_interface name="velocity"/><state_interface name="position"/><state_interface name="velocity"/></joint>
+    <joint name="iiwa2_joint_a5"><command_interface name="position"/><command_interface name="velocity"/><state_interface name="position"/><state_interface name="velocity"/></joint>
+    <joint name="iiwa2_joint_a6"><command_interface name="position"/><command_interface name="velocity"/><state_interface name="position"/><state_interface name="velocity"/></joint>
+    <joint name="iiwa2_joint_a7"><command_interface name="position"/><command_interface name="velocity"/><state_interface name="position"/><state_interface name="velocity"/></joint>
   </ros2_control>
   <gazebo>
