Commit message: backup

File: ros2_fra2mo/urdf/fra2mo_base_macro.xacro (robot description, xacro)
@@ -161,14 +161,30 @@
       </plugin>
     </gazebo>
-  <link name="container_link">
+    <link name="container_link">
       <visual>
-        <origin xyz="0 0 0.01" rpy="0 0 0" />
-        <geometry><box size="0.2 0.2 0.02"/></geometry> <material name="Blue_Dark"><color rgba="0 0 0.5 1"/></material>
+        <origin xyz="-0.1 0 0.01" rpy="0 0 0" />
+        <geometry><box size="0.4 0.4 0.02"/></geometry>
+        <material name="Blue_Dark"><color rgba="0 0 0.5 1"/></material>
       </visual>
-      <visual><origin xyz="0.095 0 0.075"/><geometry><box size="0.01 0.2 0.15"/></geometry></visual>
-      <visual><origin xyz="-0.095 0 0.075"/><geometry><box size="0.01 0.2 0.15"/></geometry></visual>
-      <visual><origin xyz="0 0.095 0.075"/><geometry><box size="0.18 0.01 0.15"/></geometry></visual>
-      <visual><origin xyz="0 -0.095 0.075"/><geometry><box size="0.18 0.01 0.15"/></geometry></visual>
-      <collision><origin xyz="0 0 0.075"/><geometry><box size="0.2 0.2 0.15"/></geometry></collision>
+      <visual>
+        <origin xyz="0.095 0 0.075"/>
+        <geometry><box size="0.01 0.4 0.15"/></geometry>
+      </visual>
+      <visual>
+        <origin xyz="-0.295 0 0.075"/>
+        <geometry><box size="0.01 0.4 0.15"/></geometry>
+      </visual>
+      <visual>
+        <origin xyz="-0.1 0.195 0.075"/>
+        <geometry><box size="0.38 0.01 0.15"/></geometry>
+      </visual>
+      <visual>
+        <origin xyz="-0.1 -0.195 0.075"/>
+        <geometry><box size="0.38 0.01 0.15"/></geometry>
+      </visual>
+      <collision>
+        <origin xyz="-0.1 0 0.075"/>
+        <geometry><box size="0.4 0.4 0.15"/></geometry>
+      </collision>
     </link>
     <joint name="container_joint" type="fixed">

File: ros2_iiwa/iiwa_description/urdf/iiwa1.urdf.xacro (robot description, xacro)
@@ -1,165 +1,193 @@
 <?xml version="1.0"?>
 <robot xmlns:xacro="http://www.ros.org/wiki/xacro" name="iiwa1">
-  <material name="gray">
-    <color rgba="0.5 0.5 0.5 1.0"/>
-  </material>
-  <link name="base_link"/>
-  <joint name="iiwa_base_joint" type="fixed">
-    <origin rpy="0.0 0 0" xyz="0 0 0"/>
-    <parent link="base_link"/>
-    <child link="iiwa_link_0"/>
-  </joint>
-  <!-- STRATEGIA: Visual = mesh (bella), Collision = primitive (veloce) -->
-  <link name="iiwa_link_0">
-    <visual>
+  <xacro:macro name="iiwa_macro" params="parent prefix *origin">
+    <material name="${prefix}gray">
+      <color rgba="0.5 0.5 0.5 1.0"/>
+    </material>
+    <link name="${prefix}iiwa_base"/>
+    <joint name="${prefix}iiwa_root_joint" type="fixed">
+      <xacro:insert_block name="origin" />
+      <parent link="${parent}"/>
+      <child link="${prefix}iiwa_base"/>
+    </joint>
+    <joint name="${prefix}iiwa_base_joint" type="fixed">
       <origin rpy="0.0 0 0" xyz="0 0 0"/>
-      <geometry><mesh filename="file://$(find iiwa_description)/meshes/lbr_iiwa_14_r820/visual/base_link.dae"/></geometry>
-    </visual>
-    <collision>
-      <!-- SOSTITUITA CON CILINDRO -->
-      <origin rpy="0 0 0" xyz="0 0 0.05"/>
-      <geometry><cylinder radius="0.08" length="0.1"/></geometry>
-    </collision>
-    <inertial>
-      <origin xyz="-0.1 0 0.07" rpy="0 0 0"/><mass value="5"/><inertia ixx="0.05" ixy="0" ixz="0" iyy="0.06" iyz="0" izz="0.03" />
-    </inertial>
-  </link>
-  <link name="iiwa_link_1">
-    <visual>
-      <geometry><mesh filename="file://$(find iiwa_description)/meshes/lbr_iiwa_14_r820/visual/link_1.dae"/></geometry>
-    </visual>
-    <collision>
-      <!-- SOSTITUITA CON CILINDRO -->
-      <origin xyz="0 0 0.18" rpy="0 0 0"/>
-      <geometry><cylinder radius="0.06" length="0.36"/></geometry>
-    </collision>
-    <inertial>
-      <origin xyz="0 -0.03 0.12" rpy="0 0 0"/><mass value="4"/><inertia ixx="0.1" ixy="0" ixz="0" iyy="0.09" iyz="0" izz="0.02" />
-    </inertial>
-  </link>
-  <link name="iiwa_link_2">
-    <visual>
-      <geometry><mesh filename="file://$(find iiwa_description)/meshes/lbr_iiwa_14_r820/visual/link_2.dae"/></geometry>
-    </visual>
-    <collision>
-      <!-- SOSTITUITA CON CILINDRO -->
-      <origin xyz="0 0.04 0" rpy="0 0 0"/>
-      <geometry><cylinder radius="0.055" length="0.1"/></geometry>
-    </collision>
-    <inertial>
-      <origin xyz="0.0003 0.059 0.042" rpy="0 0 0"/><mass value="4"/><inertia ixx="0.05" ixy="0" ixz="0" iyy="0.018" iyz="0" izz="0.044" />
-    </inertial>
-  </link>
-  <link name="iiwa_link_3">
-    <visual>
-      <geometry><mesh filename="file://$(find iiwa_description)/meshes/lbr_iiwa_14_r820/visual/link_3.dae"/></geometry>
-    </visual>
-    <collision>
-      <!-- SOSTITUITA CON CILINDRO -->
-      <origin xyz="0 0 0.21" rpy="0 0 0"/>
-      <geometry><cylinder radius="0.055" length="0.42"/></geometry>
-    </collision>
-    <inertial>
-      <origin xyz="0 0.03 0.13" rpy="0 0 0"/><mass value="3"/><inertia ixx="0.08" ixy="0" ixz="0" iyy="0.075" iyz="0" izz="0.01" />
-    </inertial>
-  </link>
-  <link name="iiwa_link_4">
-    <visual>
-      <geometry><mesh filename="file://$(find iiwa_description)/meshes/lbr_iiwa_14_r820/visual/link_4.dae"/></geometry>
-    </visual>
-    <collision>
-      <!-- SOSTITUITA CON CILINDRO -->
-      <origin xyz="0 0.04 0" rpy="0 0 0"/>
-      <geometry><cylinder radius="0.05" length="0.1"/></geometry>
-    </collision>
-    <inertial>
-      <origin xyz="0 0.067 0.034" rpy="0 0 0"/><mass value="2.7"/><inertia ixx="0.03" ixy="0" ixz="0" iyy="0.01" iyz="0" izz="0.029" />
-    </inertial>
-  </link>
-  <link name="iiwa_link_5">
-    <visual>
-      <geometry><mesh filename="file://$(find iiwa_description)/meshes/lbr_iiwa_14_r820/visual/link_5.dae"/></geometry>
-    </visual>
-    <collision>
-      <!-- SOSTITUITA CON CILINDRO -->
-      <origin xyz="0 0 0.2" rpy="0 0 0"/>
-      <geometry><cylinder radius="0.045" length="0.4"/></geometry>
-    </collision>
-    <inertial>
-      <origin xyz="0.0001 0.021 0.076" rpy="0 0 0"/><mass value="1.7"/><inertia ixx="0.02" ixy="0" ixz="0" iyy="0.018" iyz="0" izz="0.005" />
-    </inertial>
-  </link>
-  <link name="iiwa_link_6">
-    <visual>
-      <geometry><mesh filename="file://$(find iiwa_description)/meshes/lbr_iiwa_14_r820/visual/link_6.dae"/></geometry>
-    </visual>
-    <collision>
-      <!-- SOSTITUITA CON CILINDRO -->
-      <origin xyz="0 0 0" rpy="0 0 0"/>
-      <geometry><cylinder radius="0.04" length="0.08"/></geometry>
-    </collision>
-    <inertial>
-      <origin xyz="0 0.0006 0.0004" rpy="0 0 0"/><mass value="1.8"/><inertia ixx="0.025" ixy="0" ixz="0" iyy="0.0136" iyz="0" izz="0.0247" />
-    </inertial>
-  </link>
-  <link name="iiwa_link_7">
-    <visual>
-      <origin rpy="0 0 0" xyz="0 0 0.07"/>
-      <material name="gray"/>
-      <geometry><mesh filename="file://$(find iiwa_description)/meshes/lbr_iiwa_14_r820/visual/link_7_2.stl" scale="0.001 0.001 0.001"/></geometry>
-    </visual>
-    <collision>
-      <!-- SOSTITUITA CON CILINDRO -->
-      <origin rpy="0 0 0" xyz="0 0 0.077"/>
-      <geometry><cylinder radius="0.035" length="0.154"/></geometry>
-    </collision>
-    <inertial>
-      <origin xyz="0 0 0.02" rpy="0 0 0"/><mass value="0.43"/><inertia ixx="0.01" ixy="0" ixz="0" iyy="0.01" iyz="0" izz="0.01" />
-    </inertial>
-  </link>
-  <link name="iiwa_tool0"/>
-  <joint name="iiwa_joint_a1" type="revolute">
-    <origin rpy="0 0 0" xyz="0 0 0"/><parent link="iiwa_link_0"/><child link="iiwa_link_1"/><axis xyz="0 0 1"/>
-    <limit effort="320" lower="-2.9668" upper="2.9668" velocity="1.4834"/>
-    <dynamics damping="1.0" friction="0.5"/>
-  </joint>
-  <joint name="iiwa_joint_a2" type="revolute">
-    <origin rpy="0 0 0" xyz="-0.00043624 0 0.36"/><parent link="iiwa_link_1"/><child link="iiwa_link_2"/><axis xyz="0 1 0"/>
-    <limit effort="320" lower="-2.0942" upper="2.0942" velocity="1.4834"/>
-    <dynamics damping="1.0" friction="0.5"/>
-  </joint>
-  <joint name="iiwa_joint_a3" type="revolute">
-    <origin rpy="0 0 0" xyz="0 0 0"/><parent link="iiwa_link_2"/><child link="iiwa_link_3"/><axis xyz="0 0 1"/>
-    <limit effort="176" lower="-2.9668" upper="2.9668" velocity="1.7452"/>
-    <dynamics damping="1.0" friction="0.5"/>
-  </joint>
-  <joint name="iiwa_joint_a4" type="revolute">
-    <origin rpy="0 0 0" xyz="0.00043624 0 0.42"/><parent link="iiwa_link_3"/><child link="iiwa_link_4"/><axis xyz="0 -1 0"/>
-    <limit effort="176" lower="-2.0942" upper="2.0942" velocity="1.3089"/>
-    <dynamics damping="1.0" friction="0.5"/>
-  </joint>
-  <joint name="iiwa_joint_a5" type="revolute">
-    <origin rpy="0 0 0" xyz="0 0 0"/><parent link="iiwa_link_4"/><child link="iiwa_link_5"/><axis xyz="0 0 1"/>
-    <limit effort="110" lower="-2.9668" upper="2.9668" velocity="2.2688"/>
-    <dynamics damping="0.7" friction="0.3"/>
-  </joint>
-  <joint name="iiwa_joint_a6" type="revolute">
-    <origin rpy="0 0 0" xyz="0 0 0.4"/><parent link="iiwa_link_5"/><child link="iiwa_link_6"/><axis xyz="0 1 0"/>
-    <limit effort="40" lower="-2.0942" upper="2.0942" velocity="2.356"/>
-    <dynamics damping="0.7" friction="0.3"/>
-  </joint>
-  <joint name="iiwa_joint_a7" type="revolute">
-    <origin rpy="0 0 0" xyz="0 0 0"/><parent link="iiwa_link_6"/><child link="iiwa_link_7"/><axis xyz="0 0 1"/>
-    <limit effort="40" lower="-3.0541" upper="3.0541" velocity="2.356"/>
-    <dynamics damping="0.5" friction="0.2"/>
-  </joint>
-  <joint name="iiwa_joint_a7-tool0" type="fixed">
-    <origin rpy="0 0 0" xyz="0 0 0.154"/>
-    <parent link="iiwa_link_7"/>
-    <child link="iiwa_tool0"/>
-  </joint>
-  <gazebo reference="iiwa_link_7">
-    <material>Gazebo/Gray</material>
-  </gazebo>
+      <parent link="${prefix}iiwa_base"/>
+      <child link="${prefix}link_0"/>
+    </joint>
+    <link name="${prefix}link_0">
+      <visual>
+        <origin rpy="0.0 0 0" xyz="0 0 0"/>
+        <geometry><mesh filename="file://$(find iiwa_description)/meshes/lbr_iiwa_14_r820/visual/base_link.dae"/></geometry>
+      </visual>
+      <collision>
+        <origin rpy="0 0 0" xyz="0 0 0.05"/>
+        <geometry><cylinder radius="0.08" length="0.1"/></geometry>
+      </collision>
+      <inertial>
+        <origin xyz="0 0 0.05" rpy="0 0 0"/>
+        <mass value="5"/>
+        <inertia ixx="0.05" ixy="0" ixz="0" iyy="0.06" iyz="0" izz="0.03"/>
+      </inertial>
+    </link>
+    <link name="${prefix}link_1">
+      <visual>
+        <geometry><mesh filename="file://$(find iiwa_description)/meshes/lbr_iiwa_14_r820/visual/link_1.dae"/></geometry>
+      </visual>
+      <collision>
+        <origin xyz="0 0 0.01" rpy="0 0 0"/>
+        <geometry><cylinder radius="0.06" length="0.36"/></geometry>
+      </collision>-
+      <inertial>
+        <origin xyz="0 0 0.01" rpy="0 0 0"/>
+        <mass value="4"/>
+        <inertia ixx="0.05" ixy="0" ixz="0" iyy="0.05" iyz="0" izz="0.005"/>
+      </inertial>
+    </link>
+    <link name="${prefix}link_2">
+      <visual>
+        <geometry><mesh filename="file://$(find iiwa_description)/meshes/lbr_iiwa_14_r820/visual/link_2.dae"/></geometry>
+      </visual>
+      <collision>
+        <origin xyz="0 0.04 0" rpy="0 0 0"/>
+        <geometry><cylinder radius="0.055" length="0.1"/></geometry>
+      </collision>
+      <inertial>
+        <origin xyz="0 0.04 0" rpy="0 0 0"/>
+        <mass value="4"/>
+        <inertia ixx="0.04" ixy="0" ixz="0" iyy="0.005" iyz="0" izz="0.04"/>
+      </inertial>
+    </link>
+    <link name="${prefix}link_3">
+      <visual>
+        <geometry><mesh filename="file://$(find iiwa_description)/meshes/lbr_iiwa_14_r820/visual/link_3.dae"/></geometry>
+      </visual>
+      <collision>
+        <origin xyz="0 0 0.21" rpy="0 0 0"/>
+        <geometry><cylinder radius="0.055" length="0.42"/></geometry>
+      </collision>
+      <inertial>
+        <origin xyz="0 0 0.21" rpy="0 0 0"/>
+        <mass value="3"/>
+        <inertia ixx="0.06" ixy="0" ixz="0" iyy="0.06" iyz="0" izz="0.004"/>
+      </inertial>
+    </link>
+    <link name="${prefix}link_4">
+      <visual>
+        <geometry><mesh filename="file://$(find iiwa_description)/meshes/lbr_iiwa_14_r820/visual/link_4.dae"/></geometry>
+      </visual>
+      <collision>
+        <origin xyz="0 0.04 0" rpy="0 0 0"/>
+        <geometry><cylinder radius="0.05" length="0.1"/></geometry>
+      </collision>
+      <inertial>
+        <origin xyz="0 0.04 0" rpy="0 0 0"/>
+        <mass value="2.7"/>
+        <inertia ixx="0.025" ixy="0" ixz="0" iyy="0.003" iyz="0" izz="0.025"/>
+      </inertial>
+    </link>
+    <link name="${prefix}link_5">
+      <visual>
+        <geometry><mesh filename="file://$(find iiwa_description)/meshes/lbr_iiwa_14_r820/visual/link_5.dae"/></geometry>
+      </visual>
+      <collision>
+        <origin xyz="0 0 0.2" rpy="0 0 0"/>
+        <geometry><cylinder radius="0.045" length="0.4"/></geometry>
+      </collision>
+      <inertial>
+        <origin xyz="0 0 0.2" rpy="0 0 0"/>
+        <mass value="1.7"/>
+        <inertia ixx="0.03" ixy="0" ixz="0" iyy="0.03" iyz="0" izz="0.002"/>
+      </inertial>
+    </link>
+    <link name="${prefix}link_6">
+      <visual>
+        <geometry><mesh filename="file://$(find iiwa_description)/meshes/lbr_iiwa_14_r820/visual/link_6.dae"/></geometry>
+      </visual>
+      <collision>
+        <origin xyz="0 0 0" rpy="0 0 0"/>
+        <geometry><cylinder radius="0.04" length="0.08"/></geometry>
+      </collision>
+      <inertial>
+        <origin xyz="0 0 0.04" rpy="0 0 0"/>
+        <mass value="1.8"/>
+        <inertia ixx="0.015" ixy="0" ixz="0" iyy="0.015" iyz="0" izz="0.002"/>
+      </inertial>
+    </link>
+    <link name="${prefix}link_7">
+      <visual>
+        <origin rpy="0 0 0" xyz="0 0 0.07"/>
+        <geometry><mesh filename="file://$(find iiwa_description)/meshes/lbr_iiwa_14_r820/visual/link_7_2.stl" scale="0.001 0.001 0.001"/></geometry>
+        <material name="${prefix}gray"/>
+      </visual>
+      <collision>
+        <origin rpy="0 0 0" xyz="0 0 0.077"/>
+        <geometry><cylinder radius="0.035" length="0.154"/></geometry>
+      </collision>
+      <inertial>
+        <origin xyz="0 0 0.077" rpy="0 0 0"/>
+        <mass value="0.43"/>
+        <inertia ixx="0.002" ixy="0" ixz="0" iyy="0.002" iyz="0" izz="0.0005"/>
+      </inertial>
+    </link>
+    <link name="${prefix}tool0"/>
+    <joint name="${prefix}joint_a1" type="revolute">
+      <origin rpy="0 0 0" xyz="0 0 0.01"/>
+      <parent link="${prefix}link_0"/><child link="${prefix}link_1"/>
+      <axis xyz="0 0 1"/>
+      <limit effort="320" lower="-2.9668" upper="2.9668" velocity="1.4834"/>
+      <dynamics damping="5.0" friction="1.0"/>
+    </joint>
+    <joint name="${prefix}joint_a2" type="revolute">
+      <origin rpy="0 0 0" xyz="0 0 0.36"/>
+      <parent link="${prefix}link_1"/><child link="${prefix}link_2"/>
+      <axis xyz="0 1 0"/>
+      <limit effort="320" lower="-2.0942" upper="2.0942" velocity="1.4834"/>
+      <dynamics damping="5.0" friction="1.0"/>
+    </joint>
+    <joint name="${prefix}joint_a3" type="revolute">
+      <origin rpy="0 0 0" xyz="0 0 0"/>
+      <parent link="${prefix}link_2"/><child link="${prefix}link_3"/>
+      <axis xyz="0 0 1"/>
+      <limit effort="176" lower="-2.9668" upper="2.9668" velocity="1.7452"/>
+      <dynamics damping="5.0" friction="1.0"/>
+    </joint>
+    <joint name="${prefix}joint_a4" type="revolute">
+      <origin rpy="0 0 0" xyz="0 0 0.42"/>
+      <parent link="${prefix}link_3"/><child link="${prefix}link_4"/>
+      <axis xyz="0 -1 0"/>
+      <limit effort="176" lower="-2.0942" upper="2.0942" velocity="1.3089"/>
+      <dynamics damping="5.0" friction="1.0"/>
+    </joint>
+    <joint name="${prefix}joint_a5" type="revolute">
+      <origin rpy="0 0 0" xyz="0 0 0"/>
+      <parent link="${prefix}link_4"/><child link="${prefix}link_5"/>
+      <axis xyz="0 0 1"/>
+      <limit effort="110" lower="-2.9668" upper="2.9668" velocity="2.2688"/>
+      <dynamics damping="3.0" friction="0.5"/>
+    </joint>
+    <joint name="${prefix}joint_a6" type="revolute">
+      <origin rpy="0 0 0" xyz="0 0 0.4"/>
+      <parent link="${prefix}link_5"/><child link="${prefix}link_6"/>
+      <axis xyz="0 1 0"/>
+      <limit effort="40" lower="-2.0942" upper="2.0942" velocity="2.356"/>
+      <dynamics damping="3.0" friction="0.5"/>
+    </joint>
+    <joint name="${prefix}joint_a7" type="revolute">
+      <origin rpy="0 0 0" xyz="0 0 0"/>
+      <parent link="${prefix}link_6"/><child link="${prefix}link_7"/>
+      <axis xyz="0 0 1"/>
+      <limit effort="40" lower="-3.0541" upper="3.0541" velocity="2.356"/>
+      <dynamics damping="2.0" friction="0.3"/>
+    </joint>
+    <joint name="${prefix}joint_a7-tool0" type="fixed">
+      <origin rpy="0 0 0" xyz="0 0 0.154"/>
+      <parent link="${prefix}link_7"/><child link="${prefix}tool0"/>
+    </joint>
+  </xacro:macro>
+  <link name="world"/>
+  <xacro:iiwa_macro parent="world" prefix="iiwa_">
+    <origin xyz="0 0 0" rpy="0 0 0"/>
+  </xacro:iiwa_macro>
   <ros2_control name="iiwa1_hardware" type="system">
     <hardware><plugin>gz_ros2_control/GazeboSimSystem</plugin></hardware>
@@ -177,8 +205,5 @@
       <robot_param>robot_description</robot_param>
       <robot_param_node>robot_state_publisher</robot_param_node>
-      <ros>
-       <namespace>iiwa</namespace>
-       <remapping>controller_manager/robot_description:=robot_description</remapping>
-     </ros>
+      <ros><namespace>iiwa</namespace></ros>
     </plugin>
   </gazebo>
